Commit message: added *_arm_gripper_link in the URDFs for compliance with Moveit

File: dumbo_hardware_config/dumbo/urdf/dumbo.urdf.xacro (robot description, xacro)
@@ -33,5 +33,5 @@
   <xacro:dumbo_lwa name="left_arm" parent="arm_base_link" reflect="-1" />
   <!-- Schunk PG70 parallel gripper -->
-  <xacro:dumbo_pg70_gripper name="left_arm" parent="left_arm_7_link"/>
+  <xacro:dumbo_pg70_gripper name="left_arm" parent="left_arm_gripper_link"/>
   <!-- <xacro:dumbo_pg70_gripper name="right_arm" parent="right_arm_7_link"/> -->
 </robot>

File: dumbo_hardware_config/dumbo/urdf/dumbo_2grippers.urdf.xacro (robot description, xacro)
@@ -33,5 +33,5 @@
   <xacro:dumbo_lwa name="left_arm" parent="arm_base_link" reflect="-1" />
   <!-- Schunk PG70 parallel gripper -->
-  <xacro:dumbo_pg70_gripper name="left_arm" parent="left_arm_7_link"/>
-  <xacro:dumbo_pg70_gripper name="right_arm" parent="right_arm_7_link"/>
+  <xacro:dumbo_pg70_gripper name="left_arm" parent="left_arm_gripper_link"/>
+  <xacro:dumbo_pg70_gripper name="right_arm" parent="right_arm_gripper_link"/>
 </robot>

File: dumbo_hardware_config/dumbo/urdf/dumbo_robotiq.urdf.xacro (robot description, xacro)
@@ -34,9 +34,4 @@
   <xacro:dumbo_lwa name="left_arm" parent="arm_base_link" reflect="-1" />
   <!-- Schunk PG70 parallel gripper -->
-  <xacro:dumbo_pg70_gripper name="left_arm" parent="left_arm_7_link"/>
-  <!-- Schunk SDH -->
-  <xacro:schunk_sdh parent="right_arm_7_link" name="sdh">
-    <origin xyz="0.0 0.0 ${DUMBO_ARM_TIP}" rpy="0.0 0.0 ${PI}" />
-  </xacro:schunk_sdh>
-  <!-- <xacro:dumbo_pg70_gripper name="right_arm" parent="right_arm_7_link"/> -->
+  <xacro:dumbo_pg70_gripper name="left_arm" parent="left_arm_gripper_link"/>
 </robot>

File: dumbo_hardware_config/dumbo/urdf/dumbo_sdh.urdf.xacro (robot description, xacro)
@@ -34,5 +34,5 @@
   <xacro:dumbo_lwa name="left_arm" parent="arm_base_link" reflect="-1" />
   <!-- Schunk PG70 parallel gripper -->
-  <xacro:dumbo_pg70_gripper name="left_arm" parent="left_arm_7_link"/>
+  <xacro:dumbo_pg70_gripper name="left_arm" parent="left_arm_gripper_link"/>
   <!-- Schunk SDH -->
   <xacro:schunk_sdh parent="right_arm_7_link" name="sdh">

File: dumbo_hardware_config/dumbo/urdf/dumbo_vkc.urdf.xacro (robot description, xacro)
@@ -32,6 +32,6 @@
   <xacro:dumbo_lwa name="left_arm" parent="arm_base_link" reflect="-1" />
   <!-- Schunk PG70 parallel gripper -->
-  <xacro:dumbo_pg70_gripper name="left_arm" parent="left_arm_7_link"/>
-  <xacro:dumbo_pg70_gripper name="right_arm" parent="right_arm_7_link"/>
+  <xacro:dumbo_pg70_gripper name="left_arm" parent="left_arm_gripper_link"/>
+  <xacro:dumbo_pg70_gripper name="right_arm" parent="right_arm_gripper_link"/>
   <!-- VKC -->
   <xacro:dumbo_vkc name="dumbo_vkc" parent="right_arm_tool_link" child="" >

File: dumbo_hardware_config/dumbo/urdf/dumbo_vkc_new.urdf.xacro (robot description, xacro)
@@ -32,6 +32,6 @@
   <xacro:dumbo_lwa name="left_arm" parent="arm_base_link" reflect="-1" />
   <!-- Schunk PG70 parallel gripper -->
-  <xacro:dumbo_pg70_gripper name="left_arm" parent="left_arm_7_link"/>
-  <xacro:dumbo_pg70_gripper name="right_arm" parent="right_arm_7_link"/>
+  <xacro:dumbo_pg70_gripper name="left_arm" parent="left_arm_gripper_link"/>
+  <xacro:dumbo_pg70_gripper name="right_arm" parent="right_arm_gripper_link"/>
   <!-- VKC -->
   <xacro:dumbo_vkc name="dumbo_vkc" parent="right_arm_tool_link" child="" >

Commit message: Revert "added *_arm_gripper_link in the URDFs for compliance with Moveit"
This reverts commit 196b48c05d7dba58c6916886213d29b4eb98d618.

File: dumbo_hardware_config/dumbo/urdf/dumbo.urdf.xacro (robot description, xacro)
@@ -33,5 +33,5 @@
   <xacro:dumbo_lwa name="left_arm" parent="arm_base_link" reflect="-1" />
   <!-- Schunk PG70 parallel gripper -->
-  <xacro:dumbo_pg70_gripper name="left_arm" parent="left_arm_gripper_link"/>
+  <xacro:dumbo_pg70_gripper name="left_arm" parent="left_arm_7_link"/>
   <!-- <xacro:dumbo_pg70_gripper name="right_arm" parent="right_arm_7_link"/> -->
 </robot>

File: dumbo_hardware_config/dumbo/urdf/dumbo_2grippers.urdf.xacro (robot description, xacro)
@@ -33,5 +33,5 @@
   <xacro:dumbo_lwa name="left_arm" parent="arm_base_link" reflect="-1" />
   <!-- Schunk PG70 parallel gripper -->
-  <xacro:dumbo_pg70_gripper name="left_arm" parent="left_arm_gripper_link"/>
-  <xacro:dumbo_pg70_gripper name="right_arm" parent="right_arm_gripper_link"/>
+  <xacro:dumbo_pg70_gripper name="left_arm" parent="left_arm_7_link"/>
+  <xacro:dumbo_pg70_gripper name="right_arm" parent="right_arm_7_link"/>
 </robot>

File: dumbo_hardware_config/dumbo/urdf/dumbo_robotiq.urdf.xacro (robot description, xacro)
@@ -34,4 +34,9 @@
   <xacro:dumbo_lwa name="left_arm" parent="arm_base_link" reflect="-1" />
   <!-- Schunk PG70 parallel gripper -->
-  <xacro:dumbo_pg70_gripper name="left_arm" parent="left_arm_gripper_link"/>
+  <xacro:dumbo_pg70_gripper name="left_arm" parent="left_arm_7_link"/>
+  <!-- Schunk SDH -->
+  <xacro:schunk_sdh parent="right_arm_7_link" name="sdh">
+    <origin xyz="0.0 0.0 ${DUMBO_ARM_TIP}" rpy="0.0 0.0 ${PI}" />
+  </xacro:schunk_sdh>
+  <!-- <xacro:dumbo_pg70_gripper name="right_arm" parent="right_arm_7_link"/> -->
 </robot>

File: dumbo_hardware_config/dumbo/urdf/dumbo_sdh.urdf.xacro (robot description, xacro)
@@ -34,5 +34,5 @@
   <xacro:dumbo_lwa name="left_arm" parent="arm_base_link" reflect="-1" />
   <!-- Schunk PG70 parallel gripper -->
-  <xacro:dumbo_pg70_gripper name="left_arm" parent="left_arm_gripper_link"/>
+  <xacro:dumbo_pg70_gripper name="left_arm" parent="left_arm_7_link"/>
   <!-- Schunk SDH -->
   <xacro:schunk_sdh parent="right_arm_7_link" name="sdh">

File: dumbo_hardware_config/dumbo/urdf/dumbo_vkc.urdf.xacro (robot description, xacro)
@@ -32,6 +32,6 @@
   <xacro:dumbo_lwa name="left_arm" parent="arm_base_link" reflect="-1" />
   <!-- Schunk PG70 parallel gripper -->
-  <xacro:dumbo_pg70_gripper name="left_arm" parent="left_arm_gripper_link"/>
-  <xacro:dumbo_pg70_gripper name="right_arm" parent="right_arm_gripper_link"/>
+  <xacro:dumbo_pg70_gripper name="left_arm" parent="left_arm_7_link"/>
+  <xacro:dumbo_pg70_gripper name="right_arm" parent="right_arm_7_link"/>
   <!-- VKC -->
   <xacro:dumbo_vkc name="dumbo_vkc" parent="right_arm_tool_link" child="" >

File: dumbo_hardware_config/dumbo/urdf/dumbo_vkc_new.urdf.xacro (robot description, xacro)
@@ -32,6 +32,6 @@
   <xacro:dumbo_lwa name="left_arm" parent="arm_base_link" reflect="-1" />
   <!-- Schunk PG70 parallel gripper -->
-  <xacro:dumbo_pg70_gripper name="left_arm" parent="left_arm_gripper_link"/>
-  <xacro:dumbo_pg70_gripper name="right_arm" parent="right_arm_gripper_link"/>
+  <xacro:dumbo_pg70_gripper name="left_arm" parent="left_arm_7_link"/>
+  <xacro:dumbo_pg70_gripper name="right_arm" parent="right_arm_7_link"/>
   <!-- VKC -->
   <xacro:dumbo_vkc name="dumbo_vkc" parent="right_arm_tool_link" child="" >
