Commit message: fixed dumbo_robotiq urdf

File: dumbo_hardware_config/dumbo/urdf/dumbo_robotiq.urdf.xacro (robot description, xacro)
@@ -35,8 +35,3 @@
   <!-- Schunk PG70 parallel gripper -->
   <xacro:dumbo_pg70_gripper name="left_arm" parent="left_arm_7_link"/>
-  <!-- Schunk SDH -->
-  <xacro:schunk_sdh parent="right_arm_7_link" name="sdh">
-    <origin xyz="0.0 0.0 ${DUMBO_ARM_TIP}" rpy="0.0 0.0 ${PI}" />
-  </xacro:schunk_sdh>
-  <!-- <xacro:dumbo_pg70_gripper name="right_arm" parent="right_arm_7_link"/> -->
 </robot>
